File: EAGLE/ESPRemote.brd (EAGLE design)
At the start: 80 x 20 mm, 30 parts, among them U2 MCP73831, U4 3.3V

Commit message: Updated Enclosures
Parts:
- R6: value 330 -> 1k
- R9: value 10k -> 3.3k
Changed lines of the file:
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@@
 <?xml version="1.0" encoding="utf-8"?>
 <!DOCTYPE eagle SYSTEM "eagle.dtd">
-<eagle version="9.3.0">
+<eagle version="9.3.2">
 <drawing>
 <settings>
-<setting alwaysvectorfont="yes"/>
+<setting alwaysvectorfont="no"/>
 <setting verticaltext="up"/>
 </settings>
@@
 <attribute name="VALUE" x="11.557" y="19.939" size="1.27" layer="27" rot="R180"/>
 </element>
-<element name="R6" library="audio amplifier example" library_urn="urn:adsk.eagle:library:970892" package="R1206" package3d_urn="urn:adsk.eagle:package:970937/2" value="330" x="71.501" y="6.604" smashed="yes" rot="MR90">
+<element name="R6" library="audio amplifier example" library_urn="urn:adsk.eagle:library:970892" package="R1206" package3d_urn="urn:adsk.eagle:package:970937/2" value="1k" x="71.501" y="6.604" smashed="yes" rot="MR90">
 <attribute name="NAME" x="72.771" y="5.842" size="1.016" layer="26" font="vector" rot="MR90"/>
 </element>
@@
 <attribute name="VALUE" x="43.053" y="18.669" size="1.27" layer="28" rot="MR180"/>
 </element>
-<element name="R9" library="audio amplifier example" library_urn="urn:adsk.eagle:library:970892" package="R1206" package3d_urn="urn:adsk.eagle:package:970937/2" value="10k" x="44.45" y="12.7" smashed="yes" rot="MR0">
+<element name="R9" library="audio amplifier example" library_urn="urn:adsk.eagle:library:970892" package="R1206" package3d_urn="urn:adsk.eagle:package:970937/2" value="3.3k" x="44.45" y="12.7" smashed="yes" rot="MR0">
 <attribute name="NAME" x="45.085" y="10.16" size="1.016" layer="26" rot="MR0"/>
 <attribute name="VALUE" x="45.847" y="10.287" size="1.27" layer="28" rot="MR0"/>
