File: EAGLE/ESPRemote.sch (EAGLE design)
At the start: 29 parts, among them U2 MCP73831, U4 3.3V

Commit message: Updated Enclosures
Parts:
- R6: value 330 -> 1k
- R9: value 10k -> 3.3k
Changed lines of the file:
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@@
 <?xml version="1.0" encoding="utf-8"?>
 <!DOCTYPE eagle SYSTEM "eagle.dtd">
-<eagle version="9.3.0">
+<eagle version="9.3.2">
 <drawing>
 <settings>
@@
 <part name="GND1" library="SparkFun" deviceset="GND" device=""/>
 <part name="D11" library="led" library_urn="urn:adsk.eagle:library:259" deviceset="LED" device="CHIP-LED0805" package3d_urn="urn:adsk.eagle:package:15818/2" value="RED"/>
-<part name="R6" library="audio amplifier example" library_urn="urn:adsk.eagle:library:970892" deviceset="R-US_" device="R1206" package3d_urn="urn:adsk.eagle:package:970937/2" value="330"/>
+<part name="R6" library="audio amplifier example" library_urn="urn:adsk.eagle:library:970892" deviceset="R-US_" device="R1206" package3d_urn="urn:adsk.eagle:package:970937/2" value="1k"/>
 <part name="GND15" library="SparkFun" deviceset="GND" device=""/>
 <part name="GND14" library="SparkFun" deviceset="GND" device=""/>
@@
 <part name="J4" library="SparkFun-Connectors" library_urn="urn:adsk.eagle:library:9132365" deviceset="CONN_06" device="SMD-1MM" package3d_urn="urn:adsk.eagle:package:9132897/2"/>
 <part name="R8" library="audio amplifier example" library_urn="urn:adsk.eagle:library:970892" deviceset="R-US_" device="R1206" package3d_urn="urn:adsk.eagle:package:970937/2" value="10k"/>
-<part name="R9" library="audio amplifier example" library_urn="urn:adsk.eagle:library:970892" deviceset="R-US_" device="R1206" package3d_urn="urn:adsk.eagle:package:970937/2" value="10k"/>
+<part name="R9" library="audio amplifier example" library_urn="urn:adsk.eagle:library:970892" deviceset="R-US_" device="R1206" package3d_urn="urn:adsk.eagle:package:970937/2" value="3.3k"/>
 <part name="S5" library="SparkFun-Switches" library_urn="urn:adsk.eagle:library:9132704" deviceset="SWITCH-SPDT" device="-SMD-RIGHT-ANGLE" package3d_urn="urn:adsk.eagle:package:9132765/2"/>
 <part name="GND7" library="SparkFun" deviceset="GND" device=""/>
